File: My Hackpad V2.kicad_pcb (KiCad board)
At the start: 2 copper layers, 85 x 58 mm, 13 parts, among them SW1 SW_Push, SW2 SW_Push, SW3 SW_Push, SW4 SW_Push, SW5 RotaryEncoder_Switch, U1 XIAO-RP2040-DIP

Commit message: Add files via upload
Other:
- board size 85 x 58 mm -> 90 x 60 mm
- board text added: "Charles' Hackpad V2"
- board text added: "XIAO HERE!"
